Commit message: mass renaming

File: thorvald_panda_description/urdf/thorvald_model.urdf.xacro (robot description, xacro)
@@ -1,16 +1,3 @@
 <?xml version="1.0" encoding="utf-8"?>
-<!-- =================================================================================== -->
-<!-- |    This document was autogenerated by xacro from /opt/ros/melodic/share/thorvald_description/urdf/thorvald_model.xacro | -->
-<!-- |    EDITING THIS FILE BY HAND IS NOT RECOMMENDED                                 | -->
-<!-- =================================================================================== -->
-<!--
-     Maintainer: Lars Grimstad <lgrimstad@sagarobotics.com>
-     TODO
-     - config file name as arg
-     - modify to accept drive modules without steering, passive wheel modules etc.
-     - add mesh
-     - add mass properties
-     - common parameters to a config file?
--->
 <robot name="thorvald_ii">
   <gazebo>
@@ -193,64 +180,4 @@
     </actuator>
   </transmission>
-  <!-- -->
-  <!--
-    <link name="$(arg tf_prefix)rod_l_${wheel}">
-      <visual>
-        <geometry>
-          <cylinder length="20" radius="0.01"/>
-        </geometry>
-	<material name="red" />
-      </visual>
-    </link>
-    <joint name="$(arg tf_prefix)rod_l_${wheel}" type="fixed">
-      <parent link="$(arg tf_prefix)${wheel}_link"/>
-      <child link="$(arg tf_prefix)rod_l_${wheel}"/>
-      <origin xyz="0 0 10" rpy="0 0 0"/>
-      <axis xyz="0 0 1"/>
-    </joint>
-    <link name="$(arg tf_prefix)rod_r_${wheel}">
-      <visual>
-        <geometry>
-          <cylinder length="20" radius="0.01"/>
-        </geometry>
-	<material name="green" />
-      </visual>
-    </link>
-    <joint name="$(arg tf_prefix)rod_r_${wheel}" type="fixed">
-      <parent link="$(arg tf_prefix)${wheel}_link"/>
-      <child link="$(arg tf_prefix)rod_r_${wheel}"/>
-      <origin xyz="0 0 -10" rpy="0 0 0"/>
-      <axis xyz="0 0 1"/>
-    </joint>
-    <link name="$(arg tf_prefix)rod2_l_${wheel}">
-      <visual>
-        <geometry>
-          <cylinder length="80" radius="0.01"/>
-        </geometry>
-	<material name="red" />
-      </visual>
-    </link>
-    <joint name="$(arg tf_prefix)rod2_l_${wheel}" type="fixed">
-      <parent link="$(arg tf_prefix)rod_l_${wheel}"/>
-      <child link="$(arg tf_prefix)rod2_l_${wheel}"/>
-      <origin xyz="0 0 40" rpy="0 0 0"/>
-      <axis xyz="0 0 1"/>
-    </joint>
-    <link name="$(arg tf_prefix)rod2_r_${wheel}">
-      <visual>
-        <geometry>
-          <cylinder length="80" radius="0.01"/>
-        </geometry>
-	<material name="green" />
-      </visual>
-    </link>
-    <joint name="$(arg tf_prefix)rod2_r_${wheel}" type="fixed">
-      <parent link="$(arg tf_prefix)rod_r_${wheel}"/>
-      <child link="$(arg tf_prefix)rod2_r_${wheel}"/>
-      <origin xyz="0 0 -40" rpy="0 0 0"/>
-      <axis xyz="0 0 1"/>
-    </joint>
-    -->
-  <!-- -->
   <link name="top1">
     <inertial>
@@ -361,64 +288,4 @@
     </actuator>
   </transmission>
-  <!-- -->
-  <!--
-    <link name="$(arg tf_prefix)rod_l_${wheel}">
-      <visual>
-        <geometry>
-          <cylinder length="20" radius="0.01"/>
-        </geometry>
-	<material name="red" />
-      </visual>
-    </link>
-    <joint name="$(arg tf_prefix)rod_l_${wheel}" type="fixed">
-      <parent link="$(arg tf_prefix)${wheel}_link"/>
-      <child link="$(arg tf_prefix)rod_l_${wheel}"/>
-      <origin xyz="0 0 10" rpy="0 0 0"/>
-      <axis xyz="0 0 1"/>
-    </joint>
-    <link name="$(arg tf_prefix)rod_r_${wheel}">
-      <visual>
-        <geometry>
-          <cylinder length="20" radius="0.01"/>
-        </geometry>
-	<material name="green" />
-      </visual>
-    </link>
-    <joint name="$(arg tf_prefix)rod_r_${wheel}" type="fixed">
-      <parent link="$(arg tf_prefix)${wheel}_link"/>
-      <child link="$(arg tf_prefix)rod_r_${wheel}"/>
-      <origin xyz="0 0 -10" rpy="0 0 0"/>
-      <axis xyz="0 0 1"/>
-    </joint>
-    <link name="$(arg tf_prefix)rod2_l_${wheel}">
-      <visual>
-        <geometry>
-          <cylinder length="80" radius="0.01"/>
-        </geometry>
-	<material name="red" />
-      </visual>
-    </link>
-    <joint name="$(arg tf_prefix)rod2_l_${wheel}" type="fixed">
-      <parent link="$(arg tf_prefix)rod_l_${wheel}"/>
-      <child link="$(arg tf_prefix)rod2_l_${wheel}"/>
-      <origin xyz="0 0 40" rpy="0 0 0"/>
-      <axis xyz="0 0 1"/>
-    </joint>
-    <link name="$(arg tf_prefix)rod2_r_${wheel}">
-      <visual>
-        <geometry>
-          <cylinder length="80" radius="0.01"/>
-        </geometry>
-	<material name="green" />
-      </visual>
-    </link>
-    <joint name="$(arg tf_prefix)rod2_r_${wheel}" type="fixed">
-      <parent link="$(arg tf_prefix)rod_r_${wheel}"/>
-      <child link="$(arg tf_prefix)rod2_r_${wheel}"/>
-      <origin xyz="0 0 -40" rpy="0 0 0"/>
-      <axis xyz="0 0 1"/>
-    </joint>
-    -->
-  <!-- -->
   <link name="top2">
     <inertial>
@@ -529,64 +396,4 @@
     </actuator>
   </transmission>
-  <!-- -->
-  <!--
-    <link name="$(arg tf_prefix)rod_l_${wheel}">
-      <visual>
-        <geometry>
-          <cylinder length="20" radius="0.01"/>
-        </geometry>
-	<material name="red" />
-      </visual>
-    </link>
-    <joint name="$(arg tf_prefix)rod_l_${wheel}" type="fixed">
-      <parent link="$(arg tf_prefix)${wheel}_link"/>
-      <child link="$(arg tf_prefix)rod_l_${wheel}"/>
-      <origin xyz="0 0 10" rpy="0 0 0"/>
-      <axis xyz="0 0 1"/>
-    </joint>
-    <link name="$(arg tf_prefix)rod_r_${wheel}">
-      <visual>
-        <geometry>
-          <cylinder length="20" radius="0.01"/>
-        </geometry>
-	<material name="green" />
-      </visual>
-    </link>
-    <joint name="$(arg tf_prefix)rod_r_${wheel}" type="fixed">
-      <parent link="$(arg tf_prefix)${wheel}_link"/>
-      <child link="$(arg tf_prefix)rod_r_${wheel}"/>
-      <origin xyz="0 0 -10" rpy="0 0 0"/>
-      <axis xyz="0 0 1"/>
-    </joint>
-    <link name="$(arg tf_prefix)rod2_l_${wheel}">
-      <visual>
-        <geometry>
-          <cylinder length="80" radius="0.01"/>
-        </geometry>
-	<material name="red" />
-      </visual>
-    </link>
-    <joint name="$(arg tf_prefix)rod2_l_${wheel}" type="fixed">
-      <parent link="$(arg tf_prefix)rod_l_${wheel}"/>
-      <child link="$(arg tf_prefix)rod2_l_${wheel}"/>
-      <origin xyz="0 0 40" rpy="0 0 0"/>
-      <axis xyz="0 0 1"/>
-    </joint>
-    <link name="$(arg tf_prefix)rod2_r_${wheel}">
-      <visual>
-        <geometry>
-          <cylinder length="80" radius="0.01"/>
-        </geometry>
-	<material name="green" />
-      </visual>
-    </link>
-    <joint name="$(arg tf_prefix)rod2_r_${wheel}" type="fixed">
-      <parent link="$(arg tf_prefix)rod_r_${wheel}"/>
-      <child link="$(arg tf_prefix)rod2_r_${wheel}"/>
-      <origin xyz="0 0 -40" rpy="0 0 0"/>
-      <axis xyz="0 0 1"/>
-    </joint>
-    -->
-  <!-- -->
   <link name="top3">
     <inertial>
@@ -697,64 +504,4 @@
     </actuator>
   </transmission>
-  <!-- -->
-  <!--
-    <link name="$(arg tf_prefix)rod_l_${wheel}">
-      <visual>
-        <geometry>
-          <cylinder length="20" radius="0.01"/>
-        </geometry>
-	<material name="red" />
-      </visual>
-    </link>
-    <joint name="$(arg tf_prefix)rod_l_${wheel}" type="fixed">
-      <parent link="$(arg tf_prefix)${wheel}_link"/>
-      <child link="$(arg tf_prefix)rod_l_${wheel}"/>
-      <origin xyz="0 0 10" rpy="0 0 0"/>
-      <axis xyz="0 0 1"/>
-    </joint>
-    <link name="$(arg tf_prefix)rod_r_${wheel}">
-      <visual>
-        <geometry>
-          <cylinder length="20" radius="0.01"/>
-        </geometry>
-	<material name="green" />
-      </visual>
-    </link>
-    <joint name="$(arg tf_prefix)rod_r_${wheel}" type="fixed">
-      <parent link="$(arg tf_prefix)${wheel}_link"/>
-      <child link="$(arg tf_prefix)rod_r_${wheel}"/>
-      <origin xyz="0 0 -10" rpy="0 0 0"/>
-      <axis xyz="0 0 1"/>
-    </joint>
-    <link name="$(arg tf_prefix)rod2_l_${wheel}">
-      <visual>
-        <geometry>
-          <cylinder length="80" radius="0.01"/>
-        </geometry>
-	<material name="red" />
-      </visual>
-    </link>
-    <joint name="$(arg tf_prefix)rod2_l_${wheel}" type="fixed">
-      <parent link="$(arg tf_prefix)rod_l_${wheel}"/>
-      <child link="$(arg tf_prefix)rod2_l_${wheel}"/>
-      <origin xyz="0 0 40" rpy="0 0 0"/>
-      <axis xyz="0 0 1"/>
-    </joint>
-    <link name="$(arg tf_prefix)rod2_r_${wheel}">
-      <visual>
-        <geometry>
-          <cylinder length="80" radius="0.01"/>
-        </geometry>
-	<material name="green" />
-      </visual>
-    </link>
-    <joint name="$(arg tf_prefix)rod2_r_${wheel}" type="fixed">
-      <parent link="$(arg tf_prefix)rod_r_${wheel}"/>
-      <child link="$(arg tf_prefix)rod2_r_${wheel}"/>
-      <origin xyz="0 0 -40" rpy="0 0 0"/>
-      <axis xyz="0 0 1"/>
-    </joint>
-    -->
-  <!-- -->
   <link name="corner0_1">
     <inertial>

Commit message: Integrated Realsense T625 on the robot.

File: thorvald_panda_description/urdf/thorvald_model.urdf.xacro (robot description, xacro)
@@ -1,4 +1,5 @@
 <?xml version="1.0" encoding="utf-8"?>
-<robot name="thorvald_ii">
+<robot name="thorvald_ii" xmlns:xacro="http://www.ros.org/wiki/xacro">
+  <xacro:include filename="$(find realsense_t265)/urdf/_t265.urdf.xacro"/>
   <gazebo>
     <plugin filename="libthorvald_gazebo_plugins_synch.so" name="_thorvald_gazebo_plugins">
@@ -1327,3 +1328,7 @@
     </plugin>
   </gazebo>
+  <!-- Sensors. -->
+  <xacro:realsense_t265 robot_ns="thorvald/" sensor_name="t265_camera" parent_link="imu_frame" rate="30.0">
+    <origin rpy="0 0 0" xyz="0 0 0"/>
+  </xacro:realsense_t265>
 </robot>

Commit message: Added sensor l515 to thorvald robot

File: thorvald_panda_description/urdf/thorvald_model.urdf.xacro (robot description, xacro)
@@ -1,4 +1,4 @@
 <?xml version="1.0" encoding="utf-8"?>
-<robot name="thorvald_ii">
+<robot name="thorvald_ii"  xmlns:xacro="http://www.ros.org/wiki/xacro">
   <gazebo>
     <plugin filename="libthorvald_gazebo_plugins_synch.so" name="_thorvald_gazebo_plugins">
@@ -1327,3 +1327,7 @@
     </plugin>
   </gazebo>
+  <xacro:include filename="$(find realsense2_description)/urdf/_l515.urdf.xacro" />
+   <xacro:sensor_l515 name="camera" topics_ns="camera" parent="laser_frame" use_nominal_extrinsics="true" publish_pointcloud="true" add_plug="false" use_mesh="true">
+    <origin xyz="0 0 0" rpy="0 0 0" />
+  </xacro:sensor_l515>
 </robot>

Commit message: Added Lidar

File: thorvald_panda_description/urdf/thorvald_model.urdf.xacro (robot description, xacro)
@@ -1,4 +1,5 @@
 <?xml version="1.0" encoding="utf-8"?>
-<robot name="thorvald_ii">
+<robot name="thorvald_panda" xmlns:xacro="http://ros.org/wiki/xacro">
+  <xacro:arg name="laser_visual"  default="true"/>
   <gazebo>
     <plugin filename="libthorvald_gazebo_plugins_synch.so" name="_thorvald_gazebo_plugins">
@@ -69,4 +70,7 @@
     <color rgba="0.75 0.75 0.75 1"/>
   </material>
+  <material name="blue">
+    <color rgba="0.0 0.0 0.8 1.0"/>
+  </material>
   <!-- CREATE ROBOT -->
   <!-- Create base link -->
@@ -1298,4 +1302,62 @@
     <axis xyz="0 0 1"/>
   </joint>
+  <gazebo reference="base_scan">
+    <material>Gazebo/FlatBlack</material>
+    <sensor type="ray" name="lds_lfcd_sensor">
+      <pose>0.0 0 0.0 0 0 0</pose>
+      <visualize>$(arg laser_visual)</visualize>
+      <update_rate>5</update_rate>
+      <ray>
+        <scan>
+          <horizontal>
+            <samples>360</samples>
+            <resolution>1</resolution>
+            <min_angle>0.0</min_angle>
+            <max_angle>6.28319</max_angle>
+          </horizontal>
+        </scan>
+        <range>
+          <min>0.120</min>
+          <max>3.5</max>
+          <resolution>0.015</resolution>
+        </range>
+        <noise>
+          <type>gaussian</type>
+          <mean>0.0</mean>
+          <stddev>0.01</stddev>
+        </noise>
+      </ray>
+      <plugin name="gazebo_ros_lds_lfcd_controller" filename="libgazebo_ros_laser.so">
+        <topicName>scan</topicName>
+        <frameName>base_scan</frameName>
+      </plugin>
+    </sensor>
+  </gazebo>
+  <link name="base_scan">
+    <visual>
+      <origin xyz="0.0 0 0.00" rpy="0 0 0"/>
+      <geometry>
+        <mesh filename="package://thorvald_panda_description/meshes/lds.stl" scale="0.001 0.001 0.001"/>
+      </geometry>
+    </visual>
+    <collision>
+      <origin xyz="0.015 0 0.0065" rpy="0 0 0"/>
+      <geometry>
+        <cylinder length="0.0315" radius="0.055"/>
+      </geometry>
+    </collision>
+    <inertial>
+      <mass value="0.114" />
+      <origin xyz="0 0 0" />
+      <inertia ixx="0.001" ixy="0.0" ixz="0.0"
+               iyy="0.001" iyz="0.0"
+               izz="0.001" />
+    </inertial>
+  </link>
+  <joint name="scan_joint" type="fixed">
+    <parent link="base_link"/>
+    <child link="base_scan"/>
+    <origin xyz="0.664 0 0.8" rpy="0 0 0"/>
+  </joint>
   <link name="base_sensors"/>
   <link name="gps_frame"/>
